Commit message: update panda_gazebo.xarco

File: franka_description/robots/panda_gazebo.xacro (robot description, xacro)
@@ -67,5 +67,5 @@
       <child link="${arm_id}_link1"/>
       <axis xyz="0 0 1"/>
-      <limit acceleration="15" lower="-2.9671" effort="87" upper="2.9671" velocity="2.5"/>
+      <limit acceleration="15" lower="-2.8973" effort="87" upper="2.8973" velocity="2.5"/>
       <dynamics D="1" K="7000" mu_coulomb="0" mu_viscous="16" damping="0.003" friction="0.0"/>
     </joint>
@@ -97,5 +97,5 @@
       <child link="${arm_id}_link2"/>
       <axis xyz="0 0 1"/>
-      <limit acceleration="7.5" lower="-1.8326" effort="87" upper="1.8326" velocity="2.5"/>
+      <limit acceleration="7.5" lower="-1.7628" effort="87" upper="1.7628" velocity="2.5"/>
       <dynamics D="1" K="7000" mu_coulomb="0" mu_viscous="16" damping="0.003" friction="0.0"/>
     </joint>
@@ -127,5 +127,5 @@
       <child link="${arm_id}_link3"/>
       <axis xyz="0 0 1"/>
-      <limit acceleration="12.5" lower="-2.9671" effort="87" upper="2.9671" velocity="2.5"/>
+      <limit acceleration="12.5" lower="-2.8973" effort="87" upper="2.8973" velocity="2.5"/>
       <dynamics D="1" K="7000" mu_coulomb="0" mu_viscous="16" damping="0.003" friction="0.0"/>
     </joint>
@@ -157,5 +157,5 @@
       <child link="${arm_id}_link4"/>
       <axis xyz="0 0 1"/>
-      <limit acceleration="12.5" lower="-3.1416" effort="87" upper="-0.4" velocity="2.5"/>
+      <limit acceleration="12.5" lower="-3.0718" effort="87" upper="-0.0698" velocity="2.5"/>
       <dynamics D="1" K="7000" mu_coulomb="0" mu_viscous="16" damping="0.003" friction="0.0"/>
     </joint>
@@ -187,5 +187,5 @@
       <child link="${arm_id}_link5"/>
       <axis xyz="0 0 1"/>
-      <limit acceleration="15" lower="-2.9671" effort="12" upper="2.9671" velocity="3"/>
+      <limit acceleration="15" lower="-2.8973" effort="12" upper="2.8973" velocity="3"/>
       <dynamics D="1" K="7000" mu_coulomb="0" mu_viscous="16" damping="0.003" friction="0.0"/>
     </joint>
@@ -217,5 +217,5 @@
       <child link="${arm_id}_link6"/>
       <axis xyz="0 0 1"/>
-      <limit acceleration="20" lower="-0.0873" effort="12" upper="3.8223" velocity="3"/>
+      <limit acceleration="20" lower="-0.0175" effort="12" upper="3.7525" velocity="3"/>
       <dynamics D="1" K="7000" mu_coulomb="0" mu_viscous="16" damping="0.003" friction="0.0"/>
     </joint>
@@ -247,5 +247,5 @@
       <child link="${arm_id}_link7"/>
       <axis xyz="0 0 1"/>
-      <limit acceleration="20" lower="-2.9671" effort="12" upper="2.9671" velocity="3"/>
+      <limit acceleration="20" lower="-2.8973" effort="12" upper="2.8973" velocity="3"/>
       <dynamics D="1" K="7000" mu_coulomb="0" mu_viscous="16" damping="0.003" friction="0.0"/>
     </joint>
